File: Plane555/Plane555.kicad_sch (KiCad schematic)
At the start: 10 parts, among them SW1 SW_SPDT, U1 LM555xM

Commit message: feat: update board trace and R values
Other:
- note removed: "100kΩ"
Changed lines of the file:
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@@
     (effects (font (size 1.27 1.27)) (justify left bottom))
   )
-  (text "100kΩ" (at 87.63 43.18 0)
+  (text "10kΩ" (at 87.63 43.18 0)
     (effects (font (size 1.27 1.27)) (justify left bottom))
   )

Commit message: feat: update R values
Other:
- note added: "1.2kΩ"
- note added: "100kΩ"
- note added: "90Ω"
- note removed: "10kΩ"
- note removed: "220Ω"
Changed lines of the file:
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@@
     (effects (font (size 2.5 2.5)) (justify left bottom))
   )
-  (text "10kΩ" (at 101.6 55.88 0)
+  (text "100kΩ" (at 101.6 55.88 0)
     (effects (font (size 1.27 1.27)) (justify left bottom))
   )
-  (text "10kΩ" (at 87.63 43.18 0)
+  (text "1.2kΩ" (at 87.63 43.18 0)
     (effects (font (size 1.27 1.27)) (justify left bottom))
   )
-  (text "220Ω" (at 64.77 92.71 0)
+  (text "90Ω" (at 64.77 92.71 0)
     (effects (font (size 1.27 1.27)) (justify left bottom))
   )

Commit message: feat: init new files
Parts:
- D1: footprint LED_THT:LED_D3.0mm -> LED_THT:LED_D3.0mm_Horizontal_O1.27mm_Z2.0mm
- D3: footprint LED_THT:LED_D3.0mm_Horizontal_O1.27mm_Z2.0mm -> LED_THT:LED_D3.0mm
- SW1: footprint SW SS12D:Schiebeschalter SS-12D00.kicad_mod -> Button_Switch_THT:Schiebeschalter_SS-12D00
Connections:
- net +3V0: now also R2.2; no longer R1.2
- net GNDREF: now also R1.1; no longer R2.1
- net at RV1.2, U1.7 (DIS): now also R2.1; no longer R1.1
- net at D1.1 (K), D2.1 (K), D3.1 (K): now also R1.2; no longer R2.2
Other:
- title: 555 Airplane PCB with Dual Flashing LED -> Plane 555 Astable Dual LED Flasher 
